Commit message: add logic for two modes

File: my_arm.urdf (robot description, URDF)
Before this commit: robot 5dof_arm, 8 links, 7 joints
Joints:
- joint ee_joint: origin xyz=0.05 0 0 rpy=0 0 0 -> xyz=0.03 0 0 rpy=0 0 0
- joint joint3: origin xyz=-0.140 0.0 0.0 rpy=0 0 1.5707 -> xyz=-0.140 0.0 0.0 rpy=3.1416 0 2.0943
- joint joint4: origin xyz=0.105 -0.005 -0.014 rpy=-1.5707 -1.5707 -1.5707 -> xyz=0.105 0.005 0.014 rpy=-1.5707 -1.5707 -1.5707
